File: 6lekcija/Battery.kicad_pcb (KiCad board)
At the start: 2 copper layers, 2 parts

Commit message: 6Lekcijas darba pabeigshana
Parts:
- added BT3: Battery_Cell, Battery_Holders:SMTU1225-LF, F.Cu at (148.7, 119.6)
Changed lines of the file:
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@@
 (kicad_pcb (version 4) (host pcbnew 4.0.6)
   (general
-    (links 3)
-    (no_connects 3)
+    (links 5)
+    (no_connects 5)
     (area 0 0 0 0)
     (thickness 1.6)
@@
     (tracks 0)
     (zones 0)
-    (modules 2)
+    (modules 3)
     (nets 3)
   )
@@
     (mod_text_size 1 1)
     (mod_text_width 0.15)
-    (pad_size 1.524 1.524)
-    (pad_drill 0.762)
+    (pad_size 2.6 3.5)
+    (pad_drill 0)
     (pad_to_mask_clearance 0.2)
     (aux_axis_origin 0 0)
-    (visible_elements FFFFFF7F)
+    (visible_elements 7FFFFFFF)
     (pcbplotparams
       (layerselection 0x00030_80000001)
@@
       (net 1 +3V3))
   )
+  (module Battery_Holders:SMTU1225-LF (layer F.Cu)
+    (at 148.6916 119.634 180)
+    (fp_text reference BT3 (at 0 -5 180) (layer F.SilkS)
+      (effects (font (size 1 1) (thickness 0.15)))
+    )
+    (fp_text value Battery_Cell (at 0 5 180) (layer F.Fab)
+      (effects (font (size 1 1) (thickness 0.15)))
+    )
+    (pad 1 smd rect (at -10.55 0 180) (size 2.6 3.5) (layers F.Cu F.Paste F.Mask)
+      (net 1 +3V3))
+    (pad "" smd rect (at 0 0 180) (size 7 7) (layers F.Adhes))
+    (pad 2 smd rect (at 10.55 0 180) (size 2.6 3.5) (layers F.Cu F.Paste F.Mask)
+      (net 2 GND))
+  )
 )
