File: Kursa_Darbs/KursaDarbs.kicad_pcb (KiCad board)
At the start: 2 copper layers, 43 parts, among them J1 INPUT, J2 OUTPUT, J3 +40V, J4 -40V, Q1 MPSA43, Q2 MPSA43, Q3 BC546, Q4 MPSA43, Q5 BC546, Q6 MJE340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

Commit message: Kursa darba edits #2
Parts:
- moved C8 181.7 mm to (370.4, 12.6)
- moved C7 181.7 mm to (360.6, 13.6)
- moved J3 181.7 mm to (382.0, 12.1)
- moved C10 141.2 mm to (376.8, 92.0)
- moved J4 141.2 mm to (397.3, 86.9)
- moved C11 141.2 mm to (385.8, 87.8)
- moved R12 70.6 mm to (427.0, 26.8), turned to 0 degrees
- moved Q8 70.0 mm to (438.8, 22.0), turned to 0 degrees
- moved Q9 54.0 mm to (464.4, 76.2), turned to 180 degrees
- moved C6 52.6 mm to (437.1, 36.5), turned to 0 degrees
- moved R14 42.6 mm to (474.8, 38.7)
- moved D1 35.3 mm to (447.5, 30.6), turned to 180 degrees
- moved R13 35.1 mm to (469.0, 51.9)
- moved Q6 34.5 mm to (456.0, 48.3)
- moved D2 33.1 mm to (452.6, 31.8)
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Other:
- net class Power added: clearance 0.4, trace_width 18.7, via_dia 0.6, via_drill 0.4
