File: Kursa_Darbs 2/KursaDarbs.kicad_pcb (KiCad board)
At the start: 2 copper layers, 43 parts, among them J1 INPUT, J2 OUTPUT, J3 +40V, J4 -40V, Q1 MPSA43, Q2 MPSA43, Q3 BC546, Q4 MPSA43, Q5 BC546, Q6 MJE340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

Commit message: Kursa darba edits #2
Parts:
- moved J3 484.0 mm to (81.8, 65.4)
- moved J4 457.6 mm to (81.8, 113.0)
- moved C8 448.5 mm to (105.8, 64.6)
- moved C7 444.9 mm to (99.6, 65.4)
- moved C11 422.9 mm to (105.4, 117.4), turned to 90 degrees
- moved C10 419.7 mm to (99.0, 114.4), turned to 270 degrees
- moved R17 418.1 mm to (154.8, 112.7), turned to 90 degrees
- moved J2 416.1 mm to (166.4, 112.6), turned to 90 degrees
- moved C9 398.5 mm to (146.4, 113.2), turned to 270 degrees
- moved R16 392.3 mm to (146.4, 89.8)
- moved R15 392.0 mm to (136.0, 93.2)
- moved R14 382.3 mm to (136.0, 66.1)
- moved Q9 382.2 mm to (138.5, 121.6), turned to 180 degrees
- moved C6 381.3 mm to (113.4, 78.6), turned to 0 degrees
- moved R12 367.9 mm to (110.0, 68.4)
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Connections:
- J1 pad 1: GND -> Net-(C1-Pad2)
- J1 pad 2: Net-(C1-Pad2) -> GND
- J4 pad 1: Net-(C10-Pad2) -> GND
- J4 pad 2: GND -> Net-(C10-Pad2)
Routing:
- net Net-(C7-Pad1): track 0.00 -> 70.3 mm
- net Net-(C10-Pad2): track 0.00 -> 68.9 mm
- net Net-(C6-Pad2): track 0.00 -> 59.5 mm
- net Net-(Q9-Pad1): track 0.00 -> 29.3 mm
- net Net-(R14-Pad2): track 0.00 -> 25.6 mm
- net Net-(C6-Pad1): track 0.00 -> 21.0 mm
- net Net-(C3-Pad1): track 0.00 -> 20.3 mm
- net Net-(Q8-Pad3): track 0.00 -> 18.1 mm
- net Net-(C5-Pad1): track 0.00 -> 17.3 mm
- net Net-(Q3-Pad2): track 0.00 -> 15.7 mm
- net Net-(Q3-Pad1): track 0.00 -> 15.7 mm
- net Net-(Q1-Pad3): track 0.00 -> 15.4 mm
- net Net-(Q1-Pad1): track 0.00 -> 14.6 mm
- net Net-(Q5-Pad2): track 0.00 -> 12.3 mm
- net Net-(J2-Pad1): track 0.00 -> 11.6 mm
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Other:
- net class Default: clearance 0.2 -> 0.3; trace_width 0.25 -> 0.5
- net class Power added: clearance 0.4, trace_width 1.5, via_dia 0.6, via_drill 0.4
- net class highsignal added: clearance 0.6, trace_width 2.75, via_dia 0.6, via_drill 0.4
- net class lowsignal added: clearance 0.25, trace_width 0.25, via_dia 0.6, via_drill 0.4
- net class medSignal added: clearance 0.3, trace_width 1, via_dia 0.6, via_drill 0.4
- rule trace_clearance: 0.2 -> 0.3
- rule trace_min: 0.2 -> 0.1
- rule via_min_drill: 0.3 -> 0.2
- rule via_min_size: 0.4 -> 0.35

Commit message: Kursa Darbs done
Routing:
- net Net-(Q1-Pad3): track 15.4 -> 13.0 mm
- net Net-(Q5-Pad2): track 12.3 -> 10.6 mm
- net Net-(Q1-Pad1): track 14.6 -> 16.0 mm
- net Net-(C6-Pad2): track 59.5 -> 58.7 mm
- net Net-(C5-Pad1): track 17.3 -> 18.0 mm
- added copper zone on B.Cu, net GND
- added copper zone on F.Cu, net GND
Other:
- board outline added: 100.6 x 66.6 mm
- rule trace_min: 0.1 -> 0.15
- board text added: "+"
- board text added: "+40V"
- board text added: "-"
- board text added: "-40V"
- board text added: "Datorizētā projektēšana Kursa darbs: 60w Audio astiprinātājs Autors: Kristaps Vilcans"
- board text added: "Gnd"
- board text added: "IN"
- board text added: "OUT"
